Commit message: URDF Correction
Moving the origin point to the middle of the frame

File: src/robot_files/urdf/robot_files.urdf (robot description, URDF)
Before this commit: robot robot_files, 5 links, 4 joints
Joints:
- joint Left_Shoulder: origin xyz=-0.0312634311502634 -0.250000000000026 0.0527377900304119 rpy=1.57079632679489 -1.55108057106202 0 -> xyz=0.0429916429836921 0.000847722574171199 0 rpy=0 0 0
- joint Right_Shoulder: origin xyz=-0.0312634311502634 -0.250000000000026 -0.0332622099695881 rpy=1.5707963267949 -1.4632220790184 0 -> xyz=-0.0429916429836921 -0.000847722574171192 0 rpy=0 0 -0.0878584920436265

Commit message: URDF and mech.rviz updated
updated

File: src/robot_files/urdf/robot_files.urdf (robot description, URDF)
Before this commit: robot robot_files, 5 links, 4 joints
Links:
- added link Pusher, mass 0.00327033697743112; collision mesh filename=package://robot_files/meshes/Pusher.STL; visual mesh filename=package://robot_files/meshes/Pusher.STL
- link Left_Arm: mass 0.00844565667479036 -> 0.0516413964304408
- link Left_Wing: mass 0.0210754932260796 -> 0.0170525154200708
- link Right_Arm: mass 0.0123490093632538 -> 0.00787461829731969
- link Right_Wing: mass 0.0176121386529091 -> 0.0205159397398244
- link base_link: mass 0.345685675411138 -> 0.607299787326349
Joints:
- added joint Pusher_Linear_Joint: type prismatic, parent Left_Arm, child Pusher, origin xyz=0.001599 0.06201 0.080314 rpy=0 0 3.1416, axis 0 0 1, limit lower=0 upper=0.01 effort=0 velocity=0
- joint Left_Elbow: origin xyz=0 0.06 0.0328000000000001 rpy=0 0 0.762967724097882 -> xyz=0 0.06 0.0218 rpy=0 0 1.25190781692008
- joint Left_Shoulder: origin xyz=0.0429916429836921 0.000847722574171199 0 rpy=0 0 0 -> xyz=-0.057 0 0 rpy=3.14159265358979 0 -3.14147418503337
- joint Right_Elbow: origin xyz=0 0.0600000000000001 0.0218 rpy=0 0 -0.62527281558488 -> xyz=0 0.0599999999999979 0.0327999999999994 rpy=0 0 -1.22102267702235
- joint Right_Shoulder: origin xyz=-0.0429916429836921 -0.000847722574171192 0 rpy=0 0 -0.0878584920436265 -> xyz=0.057 0 0 rpy=3.14159265358979 0 3.14123293721384

Commit message: urdf axis correction
left_shoulder and left_elbow inverted along z axis

File: src/robot_files/urdf/robot_files.urdf (robot description, URDF)
Before this commit: robot robot_files, 6 links, 5 joints
Joints:
- joint Left_Elbow: axis 0 0 1 -> 0 0 -1
- joint Left_Shoulder: axis 0 0 1 -> 0 0 -1

Commit message: URDF right_elbow and left_elbow angles updated

File: src/robot_files/urdf/robot_files.urdf (robot description, URDF)
Before this commit: robot robot_files, 6 links, 5 joints
Joints:
- joint Left_Elbow: axis 0 0 -1 -> 0 0 1; origin xyz=0 0.06 0.0218 rpy=0 0 1.25190781692008 -> xyz=0 0.06 0.0218 rpy=0 0 0
- joint Right_Elbow: axis 0 0 1 -> 0 0 -1; origin xyz=0 0.0599999999999979 0.0327999999999994 rpy=0 0 -1.22102267702235 -> xyz=0 0.0599999999999979 0.0327999999999994 rpy=0 0 0
